File: bd845-pwb-tester/hat/kicad/hat.kicad_pcb (KiCad board)
At the start: 2 copper layers, 185 x 110 mm, 24 parts, among them J1 Conn_01x11, J2 Conn_01x11, J3 Conn_01x11, J4 Conn_01x11, J5 Conn_01x11, J6 Conn_01x13, J7 Conn_01x05, J8 Conn_01x13

Commit message: Hat board v1.0.0.
Parts:
- added D4: LED_U, LED_THT:LED_D3.0mm, F.Cu at (94.2, 51.0)
- added D5: LED_D, LED_THT:LED_D3.0mm, F.Cu at (126.0, 51.0)
- added D6: LED_L, LED_THT:LED_D3.0mm, F.Cu at (157.8, 51.0)
- added D7: LED_R, LED_THT:LED_D3.0mm, F.Cu at (189.5, 51.0)
- added D8: LED_C, LED_THT:LED_D3.0mm, F.Cu at (221.3, 51.0)
- added G***: LOGO, bluedot-library:bluedot-logo, F.Cu at (66.0, 138.0)
- added J9: Conn_01x05, Connector_PinHeader_2.54mm:PinHeader_1x05_P2.54mm_Vertical, F.Cu at (110.0, 127.4)
- added R10: 1k, Resistor_THT:R_Axial_DIN0207_L6.3mm_D2.5mm_P10.16mm_Horizontal, F.Cu at (110.8, 51.0)
- added R11: 1k, Resistor_THT:R_Axial_DIN0207_L6.3mm_D2.5mm_P10.16mm_Horizontal, F.Cu at (142.7, 51.0)
- added R12: 1k, Resistor_THT:R_Axial_DIN0207_L6.3mm_D2.5mm_P10.16mm_Horizontal, F.Cu at (174.3, 51.0)
- added R13: 1k, Resistor_THT:R_Axial_DIN0207_L6.3mm_D2.5mm_P10.16mm_Horizontal, F.Cu at (206.2, 51.0)
- added R9: 1k, Resistor_THT:R_Axial_DIN0207_L6.3mm_D2.5mm_P10.16mm_Horizontal, F.Cu at (79.0, 51.0)
- added REF**: OSHW-Logo_7.5x8mm_SilkScreen, Symbol:OSHW-Logo_7.5x8mm_SilkScreen, F.Cu at (91.0, 146.0)
- added REF**: WEEE-Logo_5.6x8mm_SilkScreen, Symbol:WEEE-Logo_5.6x8mm_SilkScreen, F.Cu at (101.0, 146.0)
- D1: value Status1 -> Run
- D2: value Status2 -> Success
- D3: value Status3 -> Fail
- moved D1 273.9 mm to (102.5, 95.0)
- moved D2 270.3 mm to (102.5, 88.0)
- moved J7 267.7 mm to (115.5, 127.4), turned to 180 degrees
- moved D3 267.3 mm to (102.5, 81.0)
- moved R8 228.0 mm to (118.1, 81.0), turned to 180 degrees
- moved R7 226.7 mm to (118.1, 88.0), turned to 180 degrees
- moved R6 226.0 mm to (118.1, 95.0), turned to 180 degrees
- moved J6 207.9 mm to (158.5, 144.5), turned to 90 degrees
- moved J8 178.6 mm to (153.8, 69.0), turned to 90 degrees
- moved R5 149.2 mm to (199.0, 135.4), turned to -90 degrees
- moved R4 146.3 mm to (203.0, 135.4), turned to -90 degrees
- moved R3 143.7 mm to (207.0, 135.4), turned to -90 degrees
- moved R2 141.2 mm to (211.0, 135.5), turned to -90 degrees
- moved R1 138.9 mm to (215.0, 135.4), turned to -90 degrees
Connections:
- net /LED_STATUS2 renamed /LED_SUCCESS
- J1 pad 6: +12V -> /+12V1_U
- J1 pad 9: +12V -> /+12V2_U
- J2 pad 6: +12V -> /+12V1_D
- J2 pad 9: +12V -> /+12V2_D
- J3 pad 6: +12V -> /+12V1_L
- J3 pad 9: +12V -> /+12V2_L
- J4 pad 6: +12V -> /+12V1_R
- J4 pad 9: +12V -> /+12V2_R
- J5 pad 6: +12V -> /+12V1_C
- J5 pad 9: +12V -> /+12V2_C
- R6 pad 1: /LED_STATUS1 -> /LED_RUN
- R8 pad 1: /LED_STATUS3 -> /LED_FAIL
- XA1 pad A0: /FL1 -> /U_OUT
- XA1 pad A1: /FL2 -> /D_OUT
- XA1 pad A10: /L_OUT -> /FL3
- XA1 pad A11: /D_OUT -> /FL4
- XA1 pad A12: /U_OUT -> /FL5
- XA1 pad A13: unconnected-(XA1-PadA13) -> /TEST
- XA1 pad A2: /FL3 -> /L_OUT
- XA1 pad A3: /FL4 -> /R_OUT
- XA1 pad A4: /FL5 -> /C_OUT
- XA1 pad A5: /TEST -> unconnected-(XA1-PadA5)
- XA1 pad A8: /C_OUT -> /FL1
- XA1 pad A9: /R_OUT -> /FL2
- XA1 pad D2: /LED_STATUS1 -> /LED_FAIL
- XA1 pad D4: /LED_STATUS3 -> /LED_RUN
Routing:
- net /C_LIGHT: track 0.00 -> 210.4 mm
- net /C_S1: track 0.00 -> 181.8 mm, vias 0 -> 1
- net /C_S2: track 0.00 -> 172.7 mm, vias 0 -> 1
- net /C_S3: track 0.00 -> 170.2 mm, vias 0 -> 1
- net /D_LIGHT: track 0.00 -> 164.1 mm, vias 0 -> 2
- net /C_S4: track 0.00 -> 161.3 mm, vias 0 -> 1
- net /R_LIGHT: track 0.00 -> 121.4 mm, vias 0 -> 2
- net /U_LIGHT: track 0.00 -> 114.6 mm, vias 0 -> 2
- net /LED_FAIL: track 0.00 -> 109.0 mm
- net /LED_SUCCESS: track 0.00 -> 107.6 mm
- net /LED_RUN: track 0.00 -> 105.9 mm
- net /U_S1: track 0.00 -> 89.9 mm, vias 0 -> 1
- net /U_S3: track 0.00 -> 88.5 mm, vias 0 -> 1
- net /U_S2: track 0.00 -> 82.5 mm, vias 0 -> 1
- net /U_S4: track 0.00 -> 80.6 mm, vias 0 -> 1
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- added copper zone on B.Cu, net GND
- added copper zone on F.Cu, net GND
Other:
- outline, holes or cut-outs redrawn
- rule pad_to_mask_clearance: 0 -> 0.05
- board text added: "BD845-PWB Tester Hat"
- board text added: "COMM"
- board text added: "bluedotarcade.com"
- board text added: "v1.0.0"
- board text removed: "PANEL CENTER"
- board text removed: "PANEL DOWN"
- board text removed: "PANEL LEFT"
- board text removed: "PANEL RIGHT"
- board text removed: "PANEL UP"
