File: bd845-pwb-tester/hat/kicad/hat.kicad_sch (KiCad schematic)
At the start: 24 parts, among them J1 Conn_01x11, J2 Conn_01x11, J3 Conn_01x11, J4 Conn_01x11, J5 Conn_01x11, J6 Conn_01x13, J7 Conn_01x05, J8 Conn_01x13

Commit message: Hat board v1.0.0.
Parts:
- added D4: LED_U, LED_THT:LED_D3.0mm, symbol Device:LED_Small
- added D5: LED_D, LED_THT:LED_D3.0mm, symbol Device:LED_Small
- added D6: LED_L, LED_THT:LED_D3.0mm, symbol Device:LED_Small
- added D7: LED_R, LED_THT:LED_D3.0mm, symbol Device:LED_Small
- added D8: LED_C, LED_THT:LED_D3.0mm, symbol Device:LED_Small
- added J9: Conn_01x05, Connector_PinHeader_2.54mm:PinHeader_1x05_P2.54mm_Vertical, symbol Connector_Generic:Conn_01x05
- added R10, R11, R12, R13, R9: 1k, Resistor_THT:R_Axial_DIN0207_L6.3mm_D2.5mm_P10.16mm_Horizontal, symbol Device:R_Small
- D1: value Status1 -> Run
- D2: value Status2 -> Success
- D3: value Status3 -> Fail
Connections:
- net +3V3: now also J9.1 (Pin_1)
- net C_LIGHT: now also D8.1 (K)
- net C_OUT: now also XA1.A4; no longer XA1.A8
- net D_LIGHT: now also D5.1 (K)
- net D_OUT: now also XA1.A1; no longer XA1.A11
- net FL1: now also XA1.A8; no longer XA1.A0
- net FL2: now also XA1.A9; no longer XA1.A1
- net FL3: now also XA1.A10; no longer XA1.A2
- net FL4: now also XA1.A11; no longer XA1.A3
- net FL5: now also XA1.A12; no longer XA1.A4
- net GND: now also J9.5 (Pin_5)
- net L_LIGHT: now also D6.1 (K)
- net L_OUT: now also XA1.A2; no longer XA1.A10
- net NRST: now also J9.2 (Pin_2)
- net R_LIGHT: now also D7.1 (K)
- net R_OUT: now also XA1.A3; no longer XA1.A9
- net SWCLK: now also J9.3 (Pin_3)
- net SWDIO: now also J9.4 (Pin_4)
- net TEST: now also XA1.A13; no longer XA1.A5
- net U_LIGHT: now also D4.1 (K)
- net U_OUT: now also XA1.A0; no longer XA1.A12
- removed net +12V: J1.6 (Pin_6), J1.9 (Pin_9), J2.6 (Pin_6), J2.9 (Pin_9), J3.6 (Pin_6), J3.9 (Pin_9), J4.6 (Pin_6), J4.9 (Pin_9), J5.6 (Pin_6), J5.9 (Pin_9)
- net LED_STATUS1 renamed LED_FAIL
- net LED_FAIL: now also R8.1; no longer R6.1
- net LED_STATUS2 renamed LED_SUCCESS
- net LED_STATUS3 renamed LED_RUN
- net LED_RUN: now also R6.1; no longer R8.1
- new net: D4.2 (A), R9.2
- new net: D8.2 (A), R13.2
- new net: D5.2 (A), R10.2
- new net: D6.2 (A), R11.2
- new net: D7.2 (A), R12.2
- new net +12V1_C: J5.6 (Pin_6), R13.1
- new net +12V1_D: J2.6 (Pin_6), R10.1
- new net +12V1_L: J3.6 (Pin_6), R11.1
- new net +12V1_R: J4.6 (Pin_6), R12.1
- new net +12V1_U: J1.6 (Pin_6), R9.1
- new net +12V2_C: J5.9 (Pin_9)
- new net +12V2_D: J2.9 (Pin_9)
- new net +12V2_L: J3.9 (Pin_9)
- new net +12V2_R: J4.9 (Pin_9)
- new net +12V2_U: J1.9 (Pin_9)
Other:
- moved on the sheet: D1, D2, D3, R1, R2, R3, R4, R5, R6, R7, R8
